File: Circuit/Coil/AutoTrigger.kicad_pcb (KiCad board)
At the start: 2 copper layers, 5 parts, among them J2 Trigger, Q1 BP103B

Commit message: [Circuit] Update circuit files to KiCAD 6's
Other:
- net class Default removed
