File: Circuit/Power/ZVS.kicad_pcb (KiCad board)
At the start: 2 copper layers, 66 x 73.7 mm, 18 parts, among them J1 12V DC in, J2 Output, Q1 IRFP250, Q2 IRFP250

Commit message: [Circuit] Update circuit files to KiCAD 6's
Other:
- net class Default removed
