File: Circuit/Sensor/VoltageSensor.kicad_pcb (KiCad board)
At the start: 2 copper layers, 40.6 x 27.9 mm, 22 parts, among them J1 From Capacitor Bank, J2 To Control, U1 LM393, U2 LM393, U3 PC817

Commit message: [Circuit] Update circuit files to KiCAD 6's
Other:
- net class Default removed
